File: organ_pedal_board/organ_pedal_board.kicad_sch (KiCad schematic)
At the start: 7 parts, among them J1 Conn_01x15_Socket, J2 Conn_01x15_Socket, U1 LM358

Commit message: Implement feature X to enhance user experience and fix bug Y in module Z
Parts:
- removed J1, J2: Conn_01x15_Socket, symbol Connector:Conn_01x15_Socket
- added U2: ~, symbol esp32Node:esp32devkitv1
- added U3: ADS1115IDGS, Package_SO:TSSOP-10_3x3mm_P0.5mm, symbol Analog_ADC:ADS1115IDGS
Connections:
- net GND: now also U2.2 (GND), U2.29 (GND), U3.1 (ADDR), U3.3 (GND)
- net pedal_signal: now reaches R2.2
- net pedal_signal: now also U3.4 (AIN0)
- new net dready: U2.15 (D23), U3.2 (ALERT/RDY)
- new net i2c_scl: U2.14 (D22), U3.10 (SCL)
- new net i2c_sda: U2.11 (D21), U3.9 (SDA)

Commit message: Implement initial structure for code changes
Parts:
- removed RV1: 10k, symbol Device:R_Potentiometer
- removed U1: LM358, symbol Amplifier_Operational:LM358
- added C2: 10uF, symbol Device:C
- added C3, C4: 1uF, symbol Device:C
- added C5: 100nF, symbol Device:C
- added J1: AudioPlug3, symbol Connector_Audio:AudioPlug3
- added JP1: EN, symbol Jumper:SolderJumper_2_Open
- added U1: LMV358, symbol Amplifier_Operational:LMV358
- added U4: AP2112K-3.3, Package_TO_SOT_SMD:SOT-23-5, symbol Regulator_Linear:AP2112K-3.3
Connections:
- net +3.3V: now also U2.30 (VIN), U3.8 (VDD), C2.1, C3.1, C4.2, C5.1, J1.R, U1.8 (V+), U4.5 (VOUT)
- net GND: now also C2.2, C3.2, C4.1, C5.2, J1.S, U1.4 (V-), U4.2 (GND)
- net pedal_out: now reaches R1.1
- net pedal_out: now also J1.T
- net at R2.1: now also U1.1, U1.2 (-)
- net at C1.1, R1.2: now also U1.3 (+)
- new net: JP1.2 (B), U4.3 (EN)
- new net 5v: JP1.1 (A), U4.1 (VIN)
- no-connect marks 0 -> 24
Other:
- moved on the sheet: C1, R1, R2, U2, U3
