File: Hardware/organ_pedal_board/organ_pedal_board.kicad_pcb (KiCad board)
At the start: 2 copper layers, 100 x 100 mm, 40 parts, among them J1 Conn_01x04, J2 NMJ6HFD2, J3 NMJ6HFD2, J4 ADS1115_conn, SW1 SW_Push, SW2 SW_Push, SW3 SW_Push, SW4 SW_Push, SW5 SW_Push, SW6 SW_Push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

Commit message: Refactor code structure for improved readability and maintainability
Parts:
- moved C6 2.50 mm to (163.5, 106.5)
- moved R10 1.67 mm to (193.5, 80.7)
- moved R11 1.67 mm to (193.5, 89.3)
- moved R12 1.67 mm to (193.5, 97.1)
- moved R13 1.67 mm to (193.4, 105.0)
- moved R14 1.67 mm to (193.3, 113.9)
- moved R7 1.67 mm to (193.5, 57.1)
- moved R8 1.67 mm to (193.5, 65.0)
- moved R9 1.67 mm to (193.5, 72.8)
- moved SW1 1.67 mm to (201.1, 55.7)
- moved SW2 1.67 mm to (201.1, 64.2)
- moved SW3 1.67 mm to (201.1, 73.0)
- moved SW4 1.67 mm to (201.1, 81.6)
- moved SW5 1.67 mm to (201.1, 90.2)
- moved SW6 1.67 mm to (201.2, 98.8)
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Routing:
- net /pedal1_raw: track 16.0 -> 20.0 mm
- net /button1: track 135.7 -> 138.6 mm
- net +3.3V: track 1.47 -> 3.97 mm
- net /pedal2_signal: track 59.0 -> 60.5 mm
- net /button2: track 79.9 -> 80.6 mm
- net /button8: track 17.1 -> 16.4 mm
- net /button7: track 26.5 -> 25.9 mm
- net /button5: track 44.4 -> 45.1 mm
- net /button4: track 54.7 -> 55.4 mm
- net /button3: track 63.8 -> 64.5 mm
- net Net-(J2-PadTN): track 12.9 -> 13.5 mm
- net Net-(J3-PadTN): track 12.5 -> 13.0 mm

Commit message: Refactor: Pedal Plug circuit
Parts:
- moved SW1 4.01 mm to (205.2, 55.8)
- moved R10 4.00 mm to (197.5, 80.7)
- moved R11 4.00 mm to (197.5, 89.3)
- moved R12 4.00 mm to (197.5, 97.1)
- moved R13 4.00 mm to (197.4, 105.0)
- moved R14 4.00 mm to (197.3, 113.9)
- moved R7 4.00 mm to (197.5, 57.1)
- moved R8 4.00 mm to (197.5, 65.0)
- moved R9 4.00 mm to (197.5, 72.8)
- moved SW2 4.00 mm to (205.1, 64.2)
- moved SW3 4.00 mm to (205.1, 73.0)
- moved SW4 4.00 mm to (205.1, 81.6)
- moved SW5 4.00 mm to (205.1, 90.2)
- moved SW6 4.00 mm to (205.2, 98.8)
- moved SW7 4.00 mm to (205.2, 107.4)
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Routing:
- net /button3: track 64.5 -> 68.7 mm
- net /button6: track 34.1 -> 38.1 mm
- net /button5: track 45.1 -> 49.1 mm
- net /button4: track 55.4 -> 59.4 mm
- net /button2: track 80.6 -> 84.6 mm
Other:
- board text removed: "Juntos pela música sacra"
