File: Hardware/organ_pedal_board/organ_pedal_board.kicad_pcb (KiCad board)
At the start: 2 copper layers, 100 x 100 mm, 40 parts, among them J1 Conn_01x04, J2 NMJ6HFD2, J3 NMJ6HFD2, J4 ADS1115_conn, SW1 SW_Push, SW2 SW_Push, SW3 SW_Push, SW4 SW_Push, SW5 SW_Push, SW6 SW_Push, SW7 SW_Push, SW8 SW_Push, SW9 SW_Push, U1 MCP6002-xSN

Commit message: Fix active layer and update junctions in organ pedal board schematic
- Changed active layer from 5 to 0 in the KiCad project file.
- Removed an unnecessary junction and added a new junction at updated coordinates.
- Adjusted wire connections to reflect new junction positions.
- Updated footprint properties for several components to ensure correct part references.
- Cleaned up redundant wire definitions to improve schematic clarity.
Parts:
- removed C1, C6: 10uF, Capacitor_THT:C_Disc_D10.5mm_W5.0mm_P10.00mm
- removed the R1 at (132.1, 91.0)
- removed R16: 10k, Resistor_THT:R_Axial_DIN0207_L6.3mm_D2.5mm_P5.08mm_Vertical
- removed R3: 1k, Resistor_THT:R_Axial_DIN0207_L6.3mm_D2.5mm_P5.08mm_Vertical
- added JP1: SolderJumper_3_Open, Jumper:SolderJumper-3_P1.3mm_Open_RoundedPad1.0x1.5mm, F.Cu at (123.0, 64.0)
- added JP2: SolderJumper_3_Open, Jumper:SolderJumper-3_P1.3mm_Open_RoundedPad1.0x1.5mm, F.Cu at (122.5, 72.2)
- added JP3: SolderJumper_3_Open, Jumper:SolderJumper-3_P1.3mm_Open_RoundedPad1.0x1.5mm, F.Cu at (184.5, 61.2)
- added JP4: SolderJumper_3_Open, Jumper:SolderJumper-3_P1.3mm_Open_RoundedPad1.0x1.5mm, F.Cu at (184.5, 65.0)
- added JP5: SolderJumper_2_Open, Jumper:SolderJumper-2_P1.3mm_Open_RoundedPad1.0x1.5mm, F.Cu at (189.5, 61.6)
- added JP6: SolderJumper_2_Open, Jumper:SolderJumper-2_P1.3mm_Open_RoundedPad1.0x1.5mm, F.Cu at (189.5, 65.2)
- added R4: 50k, Resistor_THT:R_Axial_DIN0207_L6.3mm_D2.5mm_P2.54mm_Vertical, F.Cu at (151.0, 94.0)
- C7, C8: value 200pF -> 10uF
- R1: renamed from R2; value 100R -> 1k
- R15: value 10k -> 50k; footprint Resistor_THT:R_Axial_DIN0207_L6.3mm_D2.5mm_P5.08mm_Vertical -> Resistor_THT:R_Axial_DIN0207_L6.3mm_D2.5mm_P2.54mm_Vertical
- R17: footprint Resistor_THT:R_Axial_DIN0207_L6.3mm_D2.5mm_P5.08mm_Vertical -> Resistor_THT:R_Axial_DIN0207_L6.3mm_D2.5mm_P2.54mm_Vertical
- R2: renamed from R4; value 100R -> 1k
- moved R15 6.90 mm to (130.5, 90.0), turned to 0 degrees
Connections:
- C7 pad 1: /pedal1_signal -> Net-(U1A-+)
- C8 pad 1: /pedal2_signal -> Net-(U1B-+)
- J2 pad R: +3.3V -> Net-(JP1-B)
- J2 pad T: /pedal1_raw -> Net-(JP1-A)
- J2 pad TN: Net-(J2-PadTN) -> unconnected-(J2-PadTN)
- J3 pad R: +3.3V -> Net-(JP3-B)
- J3 pad T: /pedal2_raw -> Net-(JP3-A)
- J3 pad TN: Net-(J3-PadTN) -> unconnected-(J3-PadTN)
- R1 pad 1: Net-(U1A--) -> /pedal1_raw
- R1 pad 2: /pedal1_signal -> Net-(U1A-+)
- R15 pad 1: Net-(J2-PadTN) -> +3.3V
- R15 pad 2: +3.3V -> Net-(JP6-B)
- R2 pad 1: Net-(U1B--) -> /pedal2_raw
- R2 pad 2: /pedal2_signal -> Net-(U1B-+)
- U1 pad 1: Net-(U1A--) -> /pedal1_signal
- U1 pad 2: Net-(U1A--) -> /pedal1_signal
- U1 pad 6: Net-(U1B--) -> /pedal2_signal
- U1 pad 7: Net-(U1B--) -> /pedal2_signal
Routing:
- net (no net): track 0.00 -> 57.9 mm
- net Net-(U1A--): track 40.4 -> 0.00 mm
- net /pedal1_raw: track 20.0 -> 0.00 mm
- net Net-(U1B--): track 17.5 -> 0.00 mm
- net Net-(JP3-A): track 0.00 -> 15.9 mm
- net /pedal2_raw: track 15.9 -> 0.00 mm
- net Net-(J2-PadTN): track 13.5 -> 0.00 mm
- net unconnected-(J3-PadTN): track 0.00 -> 13.0 mm
- net Net-(J3-PadTN): track 13.0 -> 0.00 mm
- net Net-(U1A-+): track 31.6 -> 24.1 mm
- net /button1: track 138.6 -> 140.5 mm
- net unconnected-(J2-PadTN): track 0.00 -> 0.58 mm
