File: Hardware/organ_pedal_board/organ_pedal_board.kicad_sch (KiCad schematic)
At the start: 38 parts, among them J1 Conn_01x04, J2 NMJ6HFD2, J3 NMJ6HFD2, J4 ADS1115_conn, SW1 SW_Push, SW2 SW_Push, SW3 SW_Push, SW4 SW_Push, SW5 SW_Push, SW6 SW_Push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

Commit message: Refactor code structure for improved readability and maintainability
Parts:
- removed C1, C6: 10uF, Capacitor_THT:C_Disc_D10.5mm_W5.0mm_P10.00mm, symbol Device:C
- removed R1: 1k, Resistor_THT:R_Axial_DIN0207_L6.3mm_D2.5mm_P5.08mm_Vertical, symbol Device:R
- added JP1, JP2, JP3, JP4: SolderJumper_3_Open, symbol Jumper:SolderJumper_3_Open
- added R4: 1M, symbol Device:R
- C7, C8: value 200pF -> 10uF
- R1: renamed from R2; value 100R -> 1k
- R15: value 10k -> 1M; footprint Resistor_THT:R_Axial_DIN0207_L6.3mm_D2.5mm_P5.08mm_Vertical -> (none)
- R16: value 10k -> 220R; footprint Resistor_THT:R_Axial_DIN0207_L6.3mm_D2.5mm_P5.08mm_Vertical -> (none)
- R2: renamed from R4; value 100R -> 1k
- R3: value 1k -> 220R; footprint Resistor_THT:R_Axial_DIN0207_L6.3mm_D2.5mm_P5.08mm_Vertical -> (none)
Connections:
- net +3.3V: now also R15.1, R3.2, R4.1; no longer J2.R, J3.R, R15.2
- net pedal1_raw: now also U1.3 (+), JP2.2 (C), R4.2; no longer J2.T
- net pedal2_raw: now also R15.2, U1.5 (+), JP3.2 (C); no longer J3.T, R3.1
- net at J3.TN: no longer R16.1
- net at J2.TN: no longer R15.1
- new net: J3.R, JP3.3 (B), JP4.3 (B)
- new net: J3.T, JP3.1 (A), JP4.1 (A)
- new net: J2.T, JP1.1 (A), JP2.1 (A)
- new net: JP1.2 (C), R3.1
- new net: J2.R, JP1.3 (B), JP2.3 (B)
- new net: JP4.2 (C), R16.1
- no-connect marks 22 -> 24
Other:
- moved on the sheet: C8, J2, J3, R2, U1B

Commit message: Refactor: Pedal Plug circuit
Parts:
- removed R16, R3: 220R, symbol Device:R
- added JP5, JP6: SolderJumper_2_Open, symbol Jumper:SolderJumper_2_Open
- R15, R4: value 1M -> 50k
Connections:
- net +3.3V: now also JP1.2 (C), JP4.2 (C)
- net pedal1_raw: now also R1.1, JP5.1 (A); no longer R4.2, U1.3 (+)
- net pedal1_signal: now also U1.1, U1.2 (-); no longer C7.1, R1.2
- net pedal2_raw: now also R2.1, JP6.1 (A); no longer R15.2, U1.5 (+)
- net pedal2_signal: now also U1.6 (-), U1.7; no longer C8.1, R2.2
- new net: JP6.2 (B), R15.2
- new net: C7.1, R1.2, U1.3 (+)
- new net: JP5.2 (B), R4.2
- new net: C8.1, R2.2, U1.5 (+)
Other:
- moved on the sheet: C7, C8, R1, R15, R2, R4, U1A, U1B, U1C
